File: shc/tiot-shc.sch (KiCad schematic (older format))
At the start: 4 parts, among them J0 Conn_01x03, U1 ESP32-DEVKITC-32D

Commit message: atualizado comunicação com mqtt pois placa reiniciava
Parts:
- removed J0: Conn_01x03, Connector:Banana_Jack_3Pin, symbol Connector_Generic:Conn_01x03
- added U?: DS18B20, Package_TO_SOT_THT:TO-92_Inline, symbol Sensor_Temperature:DS18B20
Connections:
- net +3V3: now also U?.1 (GND)
- net GND: now also U?.3 (VDD)
- net at R1.2, U1.32 (IO4): now also U?.2 (DQ)
Other:
- moved on the sheet: R1, U1
